Commit message: Changes for visualization

File: simulation/n-dof/urdf/kuka_iiwa/model3DOF.urdf (robot description, URDF)
Before this commit: robot lbr_iiwa, 8 links, 7 joints
Links:
- link lbr_iiwa_link_0: geometry collision mesh filename=kuka_iiwa/meshes/link_0.stl; visual mesh filename=kuka_iiwa/meshes/link_0.obj
- link lbr_iiwa_link_1: geometry collision mesh filename=kuka_iiwa/meshes/link_1.stl; visual mesh filename=kuka_iiwa/meshes/link_1.obj
- link lbr_iiwa_link_2: geometry collision mesh filename=kuka_iiwa/meshes/link_2.stl; visual mesh filename=kuka_iiwa/meshes/link_2.obj
- link lbr_iiwa_link_3: geometry collision mesh filename=kuka_iiwa/meshes/link_3.stl; visual mesh filename=kuka_iiwa/meshes/link_3.obj
- link lbr_iiwa_link_4: geometry collision mesh filename=kuka_iiwa/meshes/link_4.stl; visual mesh filename=kuka_iiwa/meshes/link_4.obj
- link lbr_iiwa_link_5: geometry collision mesh filename=kuka_iiwa/meshes/link_5.stl; visual mesh filename=kuka_iiwa/meshes/link_5.obj
- link lbr_iiwa_link_6: geometry collision mesh filename=kuka_iiwa/meshes/link_6.stl; visual mesh filename=kuka_iiwa/meshes/link_6.obj
- link lbr_iiwa_link_7: geometry collision mesh filename=kuka_iiwa/meshes/link_7.stl; visual mesh filename=kuka_iiwa/meshes/link_7.obj
